File: NIVARA/NIVARA.kicad_sch (KiCad schematic)
At the start: 12 parts, among them J10 PNP INPUT, J11 Screw_Terminal_01x02, J12 PNP OUTPUT, J13 Salidas AN, J16 Salida An 4-20mA, J3 Entrada An 0-10V, J4 Entrada An 0-32V, J5 Relay, J6 Entrada An 5-20mA, J7 NPN INPUT, J8 RS485, J9 NPN OUTPUT

Commit message: arreglo
Parts:
- renumbered J5 to J1, J13 to J10, J16 to J11, J11 to J12, J3 to J2, J4 to J3, J6 to J4, J8 to J5, J7 to J6, J9 to J7, J10 to J8, J12 to J9
Connections:
- net NIVARA/NPN_OUT_1: now also J7.2 (Pin_2); no longer J7.1 (Pin_1)
- net NIVARA/NPN_OUT_2: now also J7.1 (Pin_1); no longer J7.2 (Pin_2)
- net NIVARA/PNP_IN_1: now also J8.2 (Pin_2); no longer J8.1 (Pin_1)
- net NIVARA/PNP_IN_2: now also J8.1 (Pin_1); no longer J8.2 (Pin_2)
