File: NIVARA/POWER_SUPPLY.kicad_sch (KiCad schematic)
At the start: 9 parts, among them U3 AP63200WU

Commit message: arreglo
Parts:
- U3: footprint Package_TO_SOT_SMD:TSOT-23-6 -> (none)
Changed lines of the file:
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@@
 			)
 		)
-		(property "Footprint" "Package_TO_SOT_SMD:TSOT-23-6"
+		(property "Footprint" ""
 			(at 120.65 105.41 0)
 			(effects
