File: NIVARA/RELE_IN.kicad_sch (KiCad schematic)
At the start: 3 parts, among them K1 SANYOU_SRD_Form_C, K2 SANYOU_SRD_Form_C

Commit message: arreglo
Parts:
- U16: footprint Proyecto_componente:LK1802 -> Project Library:LK1802
Changed lines of the file:
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@@
 			)
 		)
-		(property "Footprint" "Proyecto_componente:LK1802"
+		(property "Footprint" "Project Library:LK1802"
 			(at 113.03 102.87 0)
 			(effects
