File: NIVARA/RS485_drivers.kicad_sch (KiCad schematic)
At the start: 4 parts

Commit message: arreglo
Parts:
- U15: footprint Proyecto_componente:RSM3485ECHT -> Project Library:RSM3485ECHT
Changed lines of the file:
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@@
 			)
 		)
-		(property "Footprint" "Proyecto_componente:RSM3485ECHT"
+		(property "Footprint" "Project Library:RSM3485ECHT"
 			(at 128.27 87.63 0)
 			(effects
