File: NIVARA/V_ANAG_OUT.kicad_sch (KiCad schematic)
At the start: 4 parts

Commit message: arreglo
Parts:
- C10, C11: footprint (none) -> Capacitor_SMD:C_0201_0603Metric
- U11: footprint (none) -> Project Library:GP8201S
Changed lines of the file:
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@@
 			)
 		)
-		(property "Footprint" ""
+		(property "Footprint" "Project Library:GP8201S"
 			(at 143.51 107.95 0)
 			(effects
@@
 			)
 		)
-		(property "Footprint" ""
+		(property "Footprint" "Capacitor_SMD:C_0201_0603Metric"
 			(at 167.64 96.8248 0)
 			(effects
@@
 			)
 		)
-		(property "Footprint" ""
+		(property "Footprint" "Capacitor_SMD:C_0201_0603Metric"
 			(at 159.0548 110.49 0)
 			(effects
