File: NIVARA/_autosave-NIVARA_estruc.kicad_sch (KiCad schematic)
At the start: 4 parts, among them U1 ESP32-S3-WROOM-1

Commit message: arreglo
Connections:
- net NPN_IN/NPN_IN_IN_1: no longer U1.19 (GPIO11/TOUCH11/ADC2_CH0/FSPID/FSPIIO5/SUBSPID), U1.20 (GPIO12/TOUCH12/ADC2_CH1/FSPICLK/FSPIIO6/SUBSPICLK), U1.22 (GPIO14/TOUCH14/ADC2_CH3/FSPIWP/FSPIDQS/SUBSPIWP)
- new net NPN_IN/NPN_IN_IN_2: U1.22 (GPIO14/TOUCH14/ADC2_CH3/FSPIWP/FSPIDQS/SUBSPIWP)
- new net RELE_IN/RELAY1_IN: U1.19 (GPIO11/TOUCH11/ADC2_CH0/FSPID/FSPIIO5/SUBSPID)
- new net RELE_IN/RELAY2_IN: U1.20 (GPIO12/TOUCH12/ADC2_CH1/FSPICLK/FSPIIO6/SUBSPICLK)
Changed lines of the file:
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@@
 	(paper "A4")
-	(junction
-		(at 182.88 121.92)
-		(diameter 0)
-		(color 0 0 0 0)
-	)
-	(junction
-		(at 185.42 119.38)
-		(diameter 0)
-		(color 0 0 0 0)
-	)
 	(junction
 		(at 62.23 99.06)
@@
 	)
 	(junction
-		(at 185.42 116.84)
-		(diameter 0)
-		(color 0 0 0 0)
-	)
-	(junction
-		(at 184.15 119.38)
-		(diameter 0)
-		(color 0 0 0 0)
-	)
-	(junction
 		(at 62.23 71.12)
 		(diameter 0)
 		(color 0 0 0 0)
 	)
-	(junction
-		(at 185.42 121.92)
-		(diameter 0)
-		(color 0 0 0 0)
-	)
 	(wire
 		(pts
@@
 	(wire
 		(pts
-			(xy 185.42 119.38) (xy 185.42 121.92)
-		)
-		(stroke
-			(width 0)
-			(type default)
-		)
-	)
-	(wire
-		(pts
-			(xy 187.96 146.05) (xy 187.96 121.92)
-		)
-		(stroke
-			(width 0)
-			(type default)
-		)
-	)
-	(wire
-		(pts
 			(xy 22.86 71.12) (xy 26.67 71.12)
 		)
@@
 	(wire
 		(pts
-			(xy 182.88 127) (xy 161.29 127)
-		)
-		(stroke
-			(width 0)
-			(type default)
-		)
-	)
-	(wire
-		(pts
 			(xy 166.37 147.32) (xy 166.37 132.08)
 		)
@@
 	(wire
 		(pts
-			(xy 184.15 124.46) (xy 161.29 124.46)
-		)
-		(stroke
-			(width 0)
-			(type default)
-		)
-	)
-	(wire
-		(pts
 			(xy 236.22 132.08) (xy 241.3 132.08)
 		)
@@
 	(wire
 		(pts
-			(xy 185.42 119.38) (xy 190.5 119.38)
-		)
-		(stroke
-			(width 0)
-			(type default)
-		)
-	)
-	(wire
-		(pts
 			(xy 195.58 82.55) (xy 195.58 114.3)
 		)
@@
 	(wire
 		(pts
+			(xy 175.26 120.65) (xy 175.26 127)
+		)
+		(stroke
+			(width 0)
+			(type default)
+		)
+	)
+	(wire
+		(pts
 			(xy 163.83 139.7) (xy 161.29 139.7)
 		)
@@
 	(wire
 		(pts
-			(xy 185.42 121.92) (xy 182.88 121.92)
-		)
-		(stroke
-			(width 0)
-			(type default)
-		)
-	)
-	(wire
-		(pts
 			(xy 236.22 78.74) (xy 236.22 88.9)
 		)
@@
 	(wire
 		(pts
-			(xy 185.42 116.84) (xy 185.42 119.38)
-		)
-		(stroke
-			(width 0)
-			(type default)
-		)
-	)
-	(wire
-		(pts
 			(xy 234.95 81.28) (xy 234.95 93.98)
 		)
@@
 	(wire
 		(pts
+			(xy 182.88 116.84) (xy 196.85 116.84)
+		)
+		(stroke
+			(width 0)
+			(type default)
+		)
+	)
+	(wire
+		(pts
 			(xy 237.49 64.77) (xy 241.3 64.77)
 		)
@@
 	(wire
 		(pts
+			(xy 182.88 121.92) (xy 182.88 116.84)
+		)
+		(stroke
+			(width 0)
+			(type default)
+		)
+	)
+	(wire
+		(pts
 			(xy 229.87 81.28) (xy 234.95 81.28)
 		)
@@
 	(wire
 		(pts
+			(xy 187.96 124.46) (xy 187.96 146.05)
+		)
+		(stroke
+			(width 0)
+			(type default)
+		)
+	)
+	(wire
+		(pts
 			(xy 29.21 78.74) (xy 22.86 78.74)
 		)
@@
 	(wire
 		(pts
+			(xy 184.15 119.38) (xy 184.15 114.3)
+		)
+		(stroke
+			(width 0)
+			(type default)
+		)
+	)
+	(wire
+		(pts
 			(xy 173.99 99.06) (xy 161.29 99.06)
 		)
@@
 	(wire
 		(pts
+			(xy 187.96 124.46) (xy 161.29 124.46)
+		)
+		(stroke
+			(width 0)
+			(type default)
+		)
+	)
+	(wire
+		(pts
 			(xy 59.69 50.8) (xy 64.77 50.8)
 		)
@@
 	(wire
 		(pts
-			(xy 190.5 142.24) (xy 190.5 119.38)
+			(xy 190.5 142.24) (xy 190.5 120.65)
 		)
 		(stroke
@@
 	(wire
 		(pts
-			(xy 184.15 119.38) (xy 184.15 124.46)
-		)
-		(stroke
-			(width 0)
-			(type default)
-		)
-	)
-	(wire
-		(pts
-			(xy 184.15 119.38) (xy 185.42 119.38)
-		)
-		(stroke
-			(width 0)
-			(type default)
-		)
-	)
-	(wire
-		(pts
 			(xy 226.06 40.64) (xy 232.41 40.64)
 		)
@@
 	(wire
 		(pts
-			(xy 196.85 116.84) (xy 185.42 116.84)
+			(xy 184.15 114.3) (xy 195.58 114.3)
 		)
 		(stroke
@@
 	(wire
 		(pts
-			(xy 185.42 114.3) (xy 185.42 116.84)
-		)
-		(stroke
-			(width 0)
-			(type default)
-		)
-	)
-	(wire
-		(pts
 			(xy 62.23 71.12) (xy 59.69 71.12)
 		)
@@
 	(wire
 		(pts
-			(xy 187.96 121.92) (xy 185.42 121.92)
-		)
-		(stroke
-			(width 0)
-			(type default)
-		)
-	)
-	(wire
-		(pts
 			(xy 196.85 85.09) (xy 196.85 116.84)
 		)
@@
 	(wire
 		(pts
-			(xy 195.58 114.3) (xy 185.42 114.3)
-		)
-		(stroke
-			(width 0)
-			(type default)
-		)
-	)
-	(wire
-		(pts
 			(xy 73.66 66.04) (xy 73.66 62.23)
 		)
@@
 	(wire
 		(pts
+			(xy 175.26 127) (xy 161.29 127)
+		)
+		(stroke
+			(width 0)
+			(type default)
+		)
+	)
+	(wire
+		(pts
 			(xy 67.31 144.78) (xy 69.85 144.78)
 		)
@@
 	(wire
 		(pts
+			(xy 190.5 120.65) (xy 175.26 120.65)
+		)
+		(stroke
+			(width 0)
+			(type default)
+		)
+	)
+	(wire
+		(pts
 			(xy 52.07 99.06) (xy 62.23 99.06)
 		)
@@
 		)
 		(stroke
-			(width 0)
-			(type default)
-		)
-	)
-	(wire
-		(pts
-			(xy 182.88 121.92) (xy 182.88 127)
-		)
-		(stroke
