File: NIVARA/mA_OUT.kicad_sch (KiCad schematic)
At the start: 9 parts

Commit message: arreglo
Parts:
- U12: footprint Proyecto_componente:GP8303 -> Project Library:GP8303
Changed lines of the file:
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@@
 			)
 		)
-		(property "Footprint" "Proyecto_componente:GP8303"
+		(property "Footprint" "Project Library:GP8303"
 			(at 160.02 118.11 0)
 			(effects
